Commit message: Lidar gazebo visuals disabled, now robot_core is the main core of all robots, new tiny robot (from tutorial),

File: src/boxbots/description/donBarredora.xacro (robot description, xacro)
@@ -182,3 +182,27 @@
         <material>Gazebo/Black</material>
     </gazebo>
+    <!-- RAMP -->
+    <joint name="ramp_joint" type="fixed">
+        <parent link="chassis"/>
+        <child link="ramp"/>
+        <origin xyz="0.6 0 0.01"/>
+    </joint>
+    <link name="ramp">
+        <visual>
+            <geometry>
+                <mesh filename="file://$(find boxbots)/description/meshes/ramp1x1x1.dae" scale="0.24 0.4 0.2" />
+            </geometry>
+            <material name="gray"/>
+        </visual>
+        <collision>
+            <geometry>
+                <mesh filename="file://$(find boxbots)/description/meshes/ramp1x1x1.dae" scale="0.24 0.4 0.2" />
+            </geometry>
+        </collision>
+        <inertial>
+            <origin xyz="0.09909938 0.00000001 -0.00406687"/>
+            <mass value="1.00000000"/>
+            <inertia ixx="0.01520037" ixy="-0.00000000" ixz="0.00168628" iyy="0.00506596" iyz="0.00000000" izz="0.01653226"/>
+          </inertial>
+    </link>
 </robot>

File: src/boxbots/description/lidar.xacro (robot description, xacro)
@@ -28,5 +28,5 @@
         <sensor name="laser" type="ray">
             <pose> 0 0 0 0 0 0 </pose>
-            <visualize>true</visualize>
+            <visualize>false</visualize>
             <update_rate>10</update_rate>
             <ray>

File: src/boxbots/description/robot.urdf.xacro (robot description, xacro)
@@ -1,5 +1,7 @@
 <?xml version="1.0"?>
 <robot xmlns:xacro="http://www.ros.org/wiki/xacro"  name="robot">
-    <xacro:include filename="robot_core.xacro" />
+    <xacro:arg name="robot_name" default="robot_core"/>
+    <xacro:property name="robot_name" value="$(arg robot_name)"/>
+    <xacro:include filename="${robot_name}.xacro"/>
     <xacro:include filename="gazebo_control.xacro"/>
     <xacro:include filename="lidar.xacro"/>

Commit message: robot_core desing, code reuse

File: src/boxbots/description/donBarredora.xacro (robot description, xacro)
@@ -1,185 +1,5 @@
 <?xml version="1.0"?>
 <robot xmlns:xacro="http://www.ros.org/wiki/xacro">
-    <xacro:include filename="inertial_macros.xacro"/>
-    <material name="white">
-        <color rgba="1 1 1 1"/>
-    </material>
-    <material name="orange">
-        <color rgba="1 0.3 0.1 1"/>
-    </material>
-    <material name="blue">
-        <color rgba="0.2 0.2 1 1"/>
-    </material>
-    <material name="black">
-        <color rgba="0 0 0 1"/>
-    </material>
-    <material name="red">
-        <color rgba="1 0 0 1"/>
-    </material>
-    <!-- BASE LINK -->
-    <link name="base_link">
-    </link>
-    <!-- CHASSIS LINK-->
-    <joint name="chassis_joint" type="fixed">
-        <parent link="base_link"/>
-        <child link="chassis"/>
-        <origin xyz="-0.15 0 -0.05"/>
-    </joint>
-    <link name="chassis">
-        <visual>
-            <origin xyz="0.3 0 0.1"/>
-            <geometry>
-                <box size="0.6 0.4 0.2"/>
-            </geometry>
-            <material name="gray"/>
-        </visual>
-        <collision>
-            <origin xyz="0.3 0 0.1"/>
-            <geometry>
-                <box size="0.6 0.4 0.2"/>
-            </geometry>
-        </collision>
-        <xacro:inertial_box mass="3" x="0.6" y="0.4" z="0.2">
-            <origin xyz="0.3 0 0.1" rpy="0 0 0"/>
-        </xacro:inertial_box>
-    </link>
-    <gazebo reference="chassis">
-        <material>Gazebo/Gray</material>
-    </gazebo>
-    <!--LEFT WHEEL LINK-->
-    <joint name="left_wheel_joint" type="continuous">
-        <parent link="base_link"/>
-        <child link="left_wheel"/>
-        <!-- y=+(ancho/2+grosor_rueda/2)  -->
-        <origin xyz="0 0.225 0" rpy="-${pi/2} 0 0"/>
-        <axis xyz="0 0 1"/>
-    </joint>
-    <link name="left_wheel">
-        <visual>
-            <geometry>
-                <cylinder radius="0.1" length="0.05"/>
-            </geometry>
-            <material name="black"/>
-        </visual>
-        <collision>
-            <geometry>
-                <cylinder radius="0.1" length="0.05"/>
-            </geometry>
-        </collision>
-        <xacro:inertial_cylinder mass="0.2" length="0.05" radius="0.1">
-            <origin xyz="0 0 0" rpy="0 0 0"/>
-        </xacro:inertial_cylinder>
-    </link>
-    <gazebo reference="left_wheel">
-        <material>Gazebo/Black</material>
-    </gazebo>
-    <!--RIGHT WHEEL LINK-->
-    <joint name="right_wheel_joint" type="continuous">
-        <parent link="base_link"/>
-        <child link="right_wheel"/>
-        <!-- y=-(ancho/2+grosor_rueda/2)  -->
-        <origin xyz="0 -0.225 0" rpy="${pi/2} 0 0"/>
-        <axis xyz="0 0 -1"/>
-    </joint>
-    <link name="right_wheel">
-        <visual>
-            <geometry>
-                <cylinder radius="0.1" length="0.05"/>
-            </geometry>
-            <material name="black"/>
-        </visual>
-        <collision>
-            <geometry>
-                <cylinder radius="0.1" length="0.05"/>
-            </geometry>
-        </collision>
-        <xacro:inertial_cylinder mass="0.2" length="0.05" radius="0.1">
-            <origin xyz="0 0 0" rpy="0 0 0"/>
-        </xacro:inertial_cylinder>
-    </link>
-    <gazebo reference="right_wheel">
-        <material>Gazebo/Black</material>
-    </gazebo>
-    <!-- CASTER BASE LINK-->
-    <joint name="caster_base_joint" type="fixed">
-        <parent link="chassis"/>
-        <child link="caster_base"/>
-        <origin xyz="0.5 0 0"/>
-    </joint>
-    <link name="caster_base">
-        <visual>
-            <origin xyz="0 0 -0.015"/>
-            <geometry>
-                <box size="0.04 0.04 0.03"/>
-            </geometry>
-            <material name="black"/>
-        </visual>
-        <collision>
-            <origin xyz="0 0 -0.015"/>
-            <geometry>
-                <box size="0.04 0.04 0.03"/>
-            </geometry>
-        </collision>
-        <xacro:inertial_box mass="0.02" x="0.02" y="0.02" z="0.03">
-            <origin xyz="0.35 0 0.07"/>
-        </xacro:inertial_box>
-    </link>
-    <gazebo reference="caster_wheel">
-        <material>Gazebo/Black</material>
-    </gazebo>
-    <!-- CASTER WHEEL LINK-->
-    <joint name="caster_wheel_joint" type="fixed">
-        <parent link="caster_base"/>
-        <child link="caster_wheel"/>
-        <origin xyz="0 0 -0.03"/>
-    </joint>
-    <link name="caster_wheel">
-        <visual>
-            <geometry>
-                <sphere radius="0.02"/>
-            </geometry>
-            <material name="black"/>
-        </visual>
-        <collision>
-            <geometry>
-                <sphere radius="0.02"/>
-            </geometry>
-        </collision>
-        <xacro:inertial_sphere mass="0.01" radius="0.02">
-            <origin xyz="0 0 0" rpy="0 0 0"/>
-        </xacro:inertial_sphere>
-    </link>
-    <gazebo reference="caster_wheel">
-        <material>Gazebo/Black</material>
-        <mu1 value="0.001"/>
-        <mu2 value="0.001"/>
-    </gazebo>
-    <!-- LIDAR SUPPORT LINK-->
-    <joint name="lidar_support_joint" type="fixed">
-        <parent link="chassis"/>
-        <child link="lidar_support"/>
-        <origin xyz="0.15 0 0.2"/>
-    </joint>
-    <link name="lidar_support">
-        <visual>
-            <origin xyz="0 0 0.035"/>
-            <geometry>
-                <cylinder radius="0.05" length="0.07"/>
-            </geometry>
-            <material name="black"/>2
-        </visual>
-        <collision>
-            <origin xyz="0.15 0 0.035"/>
-            <geometry>
-                <cylinder radius="0.05" length="0.07"/>
-            </geometry>
-        </collision>
-        <xacro:inertial_cylinder mass="0.1" length="0.07" radius="0.05">
-            <origin xyz="0 0 0" rpy="0 0 0"/>
-        </xacro:inertial_cylinder>
-    </link>
-    <gazebo reference="lidar_support">
-        <material>Gazebo/Black</material>
-    </gazebo>
+    <xacro:include filename="robot_core.xacro"/>
     <!-- RAMP -->
     <joint name="ramp_joint" type="fixed">

File: src/boxbots/description/gazebo_control.xacro (robot description, xacro)
@@ -6,6 +6,6 @@
             <left_joint>left_wheel_joint</left_joint>
             <right_joint>right_wheel_joint</right_joint>
-            <wheel_separation>0.35</wheel_separation>
-            <wheel_diameter>0.1</wheel_diameter>
+            <wheel_separation>0.4</wheel_separation>
+            <wheel_diameter>0.2</wheel_diameter>
             <!-- Limits -->
             <max_wheel_torque>100</max_wheel_torque>

File: src/boxbots/description/lidar.xacro (robot description, xacro)
@@ -28,5 +28,5 @@
         <sensor name="laser" type="ray">
             <pose> 0 0 0 0 0 0 </pose>
-            <visualize>false</visualize>
+            <visualize>true</visualize>
             <update_rate>10</update_rate>
             <ray>

File: src/boxbots/description/robot_core.xacro (robot description, xacro)
@@ -32,5 +32,5 @@
                 <box size="0.6 0.4 0.2"/>
             </geometry>
-            <material name="gray"/>
+            <material name="grey"/>
         </visual>
         <collision>
@@ -45,5 +45,5 @@
     </link>
     <gazebo reference="chassis">
-        <material>Gazebo/Gray</material>
+        <material>Gazebo/Grey</material>
     </gazebo>
     <!--LEFT WHEEL LINK-->

Commit message: config: mapper config file, rviz_slam file added, lidar: increased lidar range to 20, urdf core: added base_footprint_link for mapping purpose, launch_sim splitted into launch_sim_joy and launch_sim (without joystick launch).

File: src/boxbots/description/donBarredora.xacro (robot description, xacro)
@@ -21,8 +21,8 @@
         </collision>
         <inertial>
-            <origin xyz="0.09909938 0.00000001 -0.00406687"/>
+            <origin xyz="0.1 0.00000000 -0.00406687"/>
             <mass value="1.00000000"/>
             <inertia ixx="0.01520037" ixy="-0.00000000" ixz="0.00168628" iyy="0.00506596" iyz="0.00000000" izz="0.01653226"/>
-          </inertial>
+        </inertial>
     </link>
 </robot>

File: src/boxbots/description/lidar.xacro (robot description, xacro)
@@ -40,5 +40,5 @@
                 <range>
                     <min>0.3</min>
-                    <max>12</max>
+                    <max>20</max>
                 </range>
             </ray>

File: src/boxbots/description/robot_core.xacro (robot description, xacro)
@@ -19,4 +19,13 @@
     <!-- BASE LINK -->
     <link name="base_link">
+    </link>
+    <!-- BASE FOOTPRINT LINK -->
+    <!-- for 2d space reference. for mapping-->
+    <joint name="base_footprint_joint" type="fixed">
+        <parent link="base_link"/>
+        <child link="base_footprint"/>
+        <origin xyz="0 0 0" rpy="0 0 0"/>
+    </joint>
+    <link name="base_footprint">
     </link>
     <!-- CHASSIS LINK-->
@@ -122,5 +131,5 @@
         </collision>
         <xacro:inertial_box mass="0.02" x="0.02" y="0.02" z="0.03">
-            <origin xyz="0.35 0 0.07"/>
+            <origin xyz="0 0 -0.015"/>
         </xacro:inertial_box>
     </link>
