Commit message: trying to fix phisics. (Is flyng)

File: src/boxbots/description/axeBot.xacro (robot description, xacro)
@@ -29,23 +29,24 @@
                 <mesh filename="file://$(find boxbots)/description/meshes/AxeBot/chassis.dae" scale="0.10 0.10 0.10"/>
             </geometry>
-            <material name="gray"/>
-        </visual>
-        <collision>
-            <geometry>
-                <mesh filename="file://$(find boxbots)/description/meshes/AxeBot/chassis.dae" scale="0.10 0.10 0.10"/>
+            <material name="green"/>
+        </visual>
+        <collision>
+            <origin xyz="0.3 0 -0.14" rpy="${pi/2} 0 ${pi/2}"/>
+            <geometry>
+                <mesh filename="file://$(find boxbots)/description/meshes/AxeBot/chassis.dae" scale="0.09 0.1 0.1"/>
             </geometry>
         </collision>
         <inertial>
-            <origin xyz="0.28599650 74.92081104 -363.40231092"/>
-            <mass value="10.00000000"/>
+            <origin xyz="0.3 0 -0.14" rpy="${pi/2} 0 ${pi/2}"/>
+            <mass value="1.00000000"/>
             <inertia ixx="1060563.74807894" ixy="-997.20714643" ixz="3526.37132554" iyy="1179332.83720922" iyz="169857.75932349" izz="412666.53274241"/>
         </inertial>
     </link>
     <gazebo reference="chassis">
-        <material>Gazebo/Gray</material>
+        <material>Gazebo/Green</material>
     </gazebo>
     <!-- LEFT WHEEL -->
     <joint name="left_wheel_joint" type="continuous">
-        <parent link="base_link"/>
+        <parent link="chassis"/>
         <child link="left_wheel"/>
         <!-- y=+(ancho/2+grosor_rueda/2)  -->
@@ -59,21 +60,22 @@
                 <mesh filename="file://$(find boxbots)/description/meshes/AxeBot/left_wheel.dae" scale="0.10 0.10 0.10"/>
             </geometry>
-            <material name="orange"/>
-        </visual>
-        <collision>
-            <geometry>
-                <mesh filename="file://$(find boxbots)/description/meshes/AxeBot/left_wheel" scale="0.10 0.10 0.10"/>
-            </geometry>
-        </collision>
-        <xacro:inertial_cylinder mass="0.2" length="0.05" radius="0.1">
-            <origin xyz="0 0 0" rpy="0 0 0"/>
+            <material name="gray"/>
+        </visual>
+        <collision>
+            <origin xyz="0.287 -0.225 -0.1427" rpy="${pi/2} 0 ${pi/2}"/>
+            <geometry>
+                <mesh filename="file://$(find boxbots)/description/meshes/AxeBot/left_wheel.dae" scale="0.10 0.10 0.10"/>
+            </geometry>
+        </collision>
+        <xacro:inertial_cylinder mass="1.0" length="0.05" radius="0.1">
+            <origin xyz="0.287 -0.225 -0.1427" rpy="${pi/2} 0 ${pi/2}"/>
         </xacro:inertial_cylinder>
     </link>
     <gazebo reference="left_wheel">
-        <material>Gazebo/Black</material>
+        <material>Gazebo/Gray</material>
     </gazebo>
     <!-- RIGHT WHEEL -->
     <joint name="right_wheel_joint" type="continuous">
-        <parent link="base_link"/>
+        <parent link="chassis"/>
         <child link="right_wheel"/>
         <!-- y=-(ancho/2+grosor_rueda/2)  -->
@@ -87,17 +89,18 @@
                 <mesh filename="file://$(find boxbots)/description/meshes/AxeBot/right_wheel.dae" scale="0.10 0.10 0.10"/>
             </geometry>
-            <material name="orange"/>
-        </visual>
-        <collision>
-            <geometry>
-                <mesh filename="file://$(find boxbots)/description/meshes/AxeBot/right_wheel" scale="0.10 0.10 0.10"/>
-            </geometry>
-        </collision>
-        <xacro:inertial_cylinder mass="0.2" length="0.05" radius="0.1">
-            <origin xyz="0 0 0" rpy="${pi/2} 0 ${pi/2}"/>
+            <material name="gray"/>
+        </visual>
+        <collision>
+            <origin xyz="0.287 0.225 -0.1427" rpy="${pi/2} 0 ${pi/2}"/>
+            <geometry>
+                <mesh filename="file://$(find boxbots)/description/meshes/AxeBot/right_wheel.dae" scale="0.10 0.10 0.10"/>
+            </geometry>
+        </collision>
+        <xacro:inertial_cylinder mass="1.0" length="0.05" radius="0.1">
+            <origin xyz="0.287 0.225 -0.1427" rpy="${pi/2} 0 ${pi/2}"/>
         </xacro:inertial_cylinder>
     </link>
     <gazebo reference="right_wheel">
-        <material>Gazebo/Black</material>
+        <material>Gazebo/Gray</material>
     </gazebo>
     <!-- BALL WHEEL -->
@@ -105,5 +108,5 @@
         <parent link="chassis"/>
         <child link="caster_wheel"/>
-        <origin xyz="0.36 0 -0.045"/>
+        <origin xyz="0.36 0 -0.08"/>
     </joint>
     <link name="caster_wheel">
@@ -116,47 +119,47 @@
         </visual>
         <collision>
+            <origin xyz="-0.06 0 -0.09" rpy="${pi/2} 0 ${pi/2}"/>
             <geometry>
                 <mesh filename="file://$(find boxbots)/description/meshes/AxeBot/ball_wheel.dae" scale="0.10 0.10 0.10"/>
             </geometry>
         </collision>
-        <xacro:inertial_sphere mass="0.01" radius="0.02">
-            <origin xyz="0 0 0" rpy="0 0 0"/>
+        <xacro:inertial_sphere mass="1.0" radius="0.02">
+            <origin xyz="-0.06 0 -0.09" rpy="${pi/2} 0 ${pi/2}"/>
         </xacro:inertial_sphere>
     </link>
     <gazebo reference="caster_wheel">
-        <material>Gazebo/Black</material>
-        <mu1 value="0.001"/>
-        <mu2 value="0.001"/>
-    </gazebo>
-    <!-- TAIL -->
-    <joint name="tail_joint" type="fixed">
-        <parent link="chassis"/>
-        <child link="tail"/>
-        <origin xyz="-0.15 0 0.25"/>
-    </joint>
-    <link name="tail">
-        <visual>
-            <origin xyz="0.4 0 -0.43" rpy="${pi/2} 0 ${pi/2}"/>
-            <geometry>
-                <mesh filename="file://$(find boxbots)/description/meshes/AxeBot/tail.dae" scale="0.10 0.10 0.10"/>
-            </geometry>
-            <material name="orange"/>
-        </visual>
-        <collision>
-            <geometry>
-                <mesh filename="file://$(find boxbots)/description/meshes/AxeBot/tail.dae" scale="0.10 0.10 0.10" />
-            </geometry>
-        </collision>
-        <inertial>
-            <origin xyz="0.00000000 511.88767315 -903.87314003"/>
-            <mass value="4.00000000"/>
-            <inertia ixx="66692.65404649" ixy="0.00000000" ixz="-0.00000000" iyy="262901.93093076" iyz="23568.08856438" izz="245071.70572291"/>
-        </inertial>
-    </link>
-    <gazebo reference="chassis_tail">
         <material>Gazebo/Orange</material>
         <mu1 value="0.001"/>
         <mu2 value="0.001"/>
     </gazebo>
+    <!-- TAIL -->
+    <joint name="tail_joint" type="fixed">
+        <parent link="chassis"/>
+        <child link="tail"/>
+        <origin xyz="-0.15 0 0.25"/>
+    </joint>
+    <link name="tail">
+        <visual>
+            <origin xyz="0.4 0 -0.43" rpy="${pi/2} 0 ${pi/2}"/>
+            <geometry>
+                <mesh filename="file://$(find boxbots)/description/meshes/AxeBot/tail.dae" scale="0.10 0.10 0.10"/>
+            </geometry>
+            <material name="orange"/>
+        </visual>
+        <collision>
+            <origin xyz="0.4 0 -0.43" rpy="${pi/2} 0 ${pi/2}"/>
+            <geometry>
+                <mesh filename="file://$(find boxbots)/description/meshes/AxeBot/tail.dae" scale="0.10 0.10 0.10"/>
+            </geometry>
+        </collision>
+        <inertial>
+            <origin xyz="0.4 0 -0.43" rpy="${pi/2} 0 ${pi/2}"/>
+            <mass value="1.00000000"/>
+            <inertia ixx="66692.65404649" ixy="0.00000000" ixz="-0.00000000" iyy="262901.93093076" iyz="23568.08856438" izz="245071.70572291"/>
+        </inertial>
+    </link>
+    <gazebo reference="chassis_tail">
+        <material>Gazebo/Orange </material>
+    </gazebo>
     <!-- AXE -->
     <joint name="axe_joint" type="fixed">
@@ -171,27 +174,26 @@
                 <mesh filename="file://$(find boxbots)/description/meshes/AxeBot/axe.dae" scale="0.10 0.10 0.10"/>
             </geometry>
-            <material name="orange"/>
-        </visual>
-        <collision>
-            <geometry>
-                <mesh filename="file://$(find boxbots)/description/meshes/AxeBot/axe.dae" scale="0.10 0.10 0.10" />
+            <material name="red"/>
+        </visual>
+        <collision>
+            <origin xyz="-0.3 0 -0.15" rpy="${pi/2} 0 ${pi/2}"/>
+            <geometry>
+                <mesh filename="file://$(find boxbots)/description/meshes/AxeBot/axe.dae" scale="0.10 0.10 0.10"/>
             </geometry>
         </collision>
         <inertial>
-            <origin xyz="-0.00097103 41.88680560 541.17520414"/>
-            <mass value="25.00000000"/>
+            <origin xyz="-0.3 0 -0.15" rpy="${pi/2} 0 ${pi/2}"/>
+            <mass value="1.00000000"/>
             <inertia ixx="544544.92866685" ixy="0.05936438" ixz="15.78266815" iyy="1117851.27450615" iyz="3282.66550122" izz="590531.59263961"/>
         </inertial>
     </link>
     <gazebo reference="axe">
-        <material>Gazebo/Orange</material>
-        <mu1 value="0.001"/>
-        <mu2 value="0.001"/>
+        <material>Gazebo/Red</material>
     </gazebo>
     <!-- LIDAR SUPPORT LINK-->
     <joint name="lidar_support_joint" type="fixed">
-        <parent link="chassis"/>
+        <parent link="tail"/>
         <child link="lidar_support"/>
-        <origin xyz="-0.18 0 0.2"/>
+        <origin xyz="-0.07 0 0"/>
     </joint>
     <link name="lidar_support">
@@ -201,8 +203,8 @@
                 <cylinder radius="0.05" length="0.07"/>
             </geometry>
-            <material name="gray"/>2
-        </visual>
-        <collision>
-            <origin xyz="0.15 0 0.035"/>
+            <material name="red"/>
+        </visual>
+        <collision>
+            <origin xyz="0 0 0.035"/>
             <geometry>
                 <cylinder radius="0.05" length="0.07"/>
@@ -210,5 +212,5 @@
         </collision>
         <xacro:inertial_cylinder mass="0.1" length="0.07" radius="0.05">
-            <origin xyz="0 0 0" rpy="0 0 0"/>
+            <origin xyz="0 0 0"/>
         </xacro:inertial_cylinder>
     </link>

Commit message: AxeBot running

File: src/boxbots/description/axeBot.xacro (robot description, xacro)
@@ -37,9 +37,7 @@
             </geometry>
         </collision>
-        <inertial>
-            <origin xyz="0.3 0 -0.14" rpy="${pi/2} 0 ${pi/2}"/>
-            <mass value="1.00000000"/>
-            <inertia ixx="1060563.74807894" ixy="-997.20714643" ixz="3526.37132554" iyy="1179332.83720922" iyz="169857.75932349" izz="412666.53274241"/>
-        </inertial>
+        <xacro:inertial_box mass="1" x="0.6" y="0.4" z="0.3">
+            <origin xyz="0.18 0 0.05" rpy="0 0 0"/>
+        </xacro:inertial_box>
     </link>
     <gazebo reference="chassis">
@@ -69,5 +67,5 @@
         </collision>
         <xacro:inertial_cylinder mass="1.0" length="0.05" radius="0.1">
-            <origin xyz="0.287 -0.225 -0.1427" rpy="${pi/2} 0 ${pi/2}"/>
+            <origin xyz="0 0 0" rpy="0 0 0"/>
         </xacro:inertial_cylinder>
     </link>
@@ -98,5 +96,5 @@
         </collision>
         <xacro:inertial_cylinder mass="1.0" length="0.05" radius="0.1">
-            <origin xyz="0.287 0.225 -0.1427" rpy="${pi/2} 0 ${pi/2}"/>
+            <origin xyz="0 0 0" rpy="0 0 0"/>
         </xacro:inertial_cylinder>
     </link>
@@ -124,6 +122,6 @@
             </geometry>
         </collision>
-        <xacro:inertial_sphere mass="1.0" radius="0.02">
-            <origin xyz="-0.06 0 -0.09" rpy="${pi/2} 0 ${pi/2}"/>
+        <xacro:inertial_sphere mass="1.0" radius="0.05">
+            <origin xyz="0 0 0" rpy="0 0 0"/>
         </xacro:inertial_sphere>
     </link>
@@ -153,9 +151,7 @@
             </geometry>
         </collision>
-        <inertial>
-            <origin xyz="0.4 0 -0.43" rpy="${pi/2} 0 ${pi/2}"/>
-            <mass value="1.00000000"/>
-            <inertia ixx="66692.65404649" ixy="0.00000000" ixz="-0.00000000" iyy="262901.93093076" iyz="23568.08856438" izz="245071.70572291"/>
-        </inertial>
+        <xacro:inertial_box mass="1" x="0.2" y="0.49" z="0.1">
+            <origin xyz="-0.04 0 -0.01" rpy="0 0 0"/>
+        </xacro:inertial_box>
     </link>
     <gazebo reference="chassis_tail">
@@ -166,5 +162,5 @@
         <parent link="chassis"/>
         <child link="axe"/>
-         <origin xyz="0.6 0 0.01"/>
+        <origin xyz="0.6 0 0.01"/>
     </joint>
     <link name="axe">
@@ -182,9 +178,7 @@
             </geometry>
         </collision>
-        <inertial>
-            <origin xyz="-0.3 0 -0.15" rpy="${pi/2} 0 ${pi/2}"/>
-            <mass value="1.00000000"/>
-            <inertia ixx="544544.92866685" ixy="0.05936438" ixz="15.78266815" iyy="1117851.27450615" iyz="3282.66550122" izz="590531.59263961"/>
-        </inertial>
+        <xacro:inertial_box mass="1" x="0.3" y="0.35" z="0.03">
+            <origin xyz="0.04 0 0" rpy="0 0 0"/>
+        </xacro:inertial_box>
     </link>
     <gazebo reference="axe">

Commit message: right wheel axis

File: src/boxbots/description/axeBot.xacro (robot description, xacro)
@@ -3,6 +3,6 @@
 <!-- Ancho: 0.3m , grosor de rueda 0.05m  Alto: 0.6m Largo: 0.6m -->
     <xacro:include filename="inertial_macros.xacro"/>
-    <material name="orange">
-        <color rgba="1 0.6 0.2 1"/>
+    <material name="white">
+        <color rgba="1 1 1 1"/>
     </material>
     <material name="green">
@@ -42,5 +42,5 @@
     </link>
     <gazebo reference="chassis">
-        <material>Gazebo/Green</material>
+        <material>Gazebo/Turquoise</material>
     </gazebo>
     <!-- LEFT WHEEL -->
@@ -79,5 +79,5 @@
         <!-- y=-(ancho/2+grosor_rueda/2)  -->
         <origin xyz="0 -0.225 0"/>
-        <axis xyz="0 -1 0"/>
+        <axis xyz="0 1 0"/>
     </joint>
     <link name="right_wheel">
@@ -114,5 +114,5 @@
                 <mesh filename="file://$(find boxbots)/description/meshes/AxeBot/ball_wheel.dae" scale="0.10 0.10 0.10"/>
             </geometry>
-            <material name="orange"/>
+            <material name="white"/>
         </visual>
         <collision>
@@ -127,5 +127,5 @@
     </link>
     <gazebo reference="caster_wheel">
-        <material>Gazebo/Orange</material>
+        <material>Gazebo/White</material>
         <mu1 value="0.001"/>
         <mu2 value="0.001"/>
@@ -143,5 +143,5 @@
                 <mesh filename="file://$(find boxbots)/description/meshes/AxeBot/tail.dae" scale="0.10 0.10 0.10"/>
             </geometry>
-            <material name="orange"/>
+            <material name="white"/>
         </visual>
         <collision>
@@ -155,6 +155,6 @@
         </xacro:inertial_box>
     </link>
-    <gazebo reference="chassis_tail">
-        <material>Gazebo/Orange </material>
+    <gazebo reference="tail">
+        <material>Gazebo/YellowGlow</material>
     </gazebo>
     <!-- AXE -->
@@ -162,5 +162,5 @@
         <parent link="chassis"/>
         <child link="axe"/>
-        <origin xyz="0.6 0 0.01"/>
+        <origin xyz="0.6 0 0.01" />
     </joint>
     <link name="axe">
@@ -183,5 +183,5 @@
     </link>
     <gazebo reference="axe">
-        <material>Gazebo/Red</material>
+        <material>Gazebo/RedGlow</material>
     </gazebo>
     <!-- LIDAR SUPPORT LINK-->

Commit message: lidar orizontal

File: src/boxbots/description/axeBot.xacro (robot description, xacro)
@@ -106,5 +106,5 @@
         <parent link="chassis"/>
         <child link="caster_wheel"/>
-        <origin xyz="0.36 0 -0.08"/>
+        <origin xyz="0.36 0 -0.045"/>
     </joint>
     <link name="caster_wheel">

Commit message: fixing control axeBot with joystick

File: src/boxbots/description/axeBot.xacro (robot description, xacro)
@@ -1,5 +1,4 @@
 <?xml version="1.0"?>
 <robot xmlns:xacro="http://www.ros.org/wiki/xacro">
-<!-- Ancho: 0.3m , grosor de rueda 0.05m  Alto: 0.6m Largo: 0.6m -->
     <xacro:include filename="inertial_macros.xacro"/>
     <material name="orange">

File: src/boxbots/description/ros2_control.xacro (robot description, xacro)
@@ -1,57 +1,25 @@
 <?xml version="1.0"?>
 <robot xmlns:xacro="http://www.ros.org/wiki/xacro">
-    <xacro:unless value="$(arg sim_mode)">
-        <ros2_control name="RealRobot" type="system">
-            <hardware>
-                <plugin>diffdrive_arduino/DiffDriveArduino</plugin>
-                <param name="left_wheel_name">left_wheel_joint</param>
-                <param name="right_wheel_name">right_wheel_joint</param>
-                <param name="loop_rate">30</param>
-                <param name="device">/dev/ttyUSB0</param>
-                <param name="baud_rate">57600</param>
-                <param name="timeout">1000</param>
-                <param name="enc_counts_per_rev">3436</param>
-            </hardware>
-            <joint name="left_wheel_joint">
-                <command_interface name="velocity">
-                    <param name="min">-10</param>
-                    <param name="max">10</param>
-                </command_interface>
-                <state_interface name="velocity"/>
-                <state_interface name="position"/>
-            </joint>
-            <joint name="right_wheel_joint">
-                <command_interface name="velocity">
-                    <param name="min">-10</param>
-                    <param name="max">10</param>
-                </command_interface>
-                <state_interface name="velocity"/>
-                <state_interface name="position"/>
-            </joint>
-        </ros2_control>
-    </xacro:unless>
-    <xacro:if value="$(arg sim_mode)">
-        <ros2_control name="GazeboSystem" type="system">
-            <hardware>
-                <plugin>gazebo_ros2_control/GazeboSystem</plugin>
-            </hardware>
-            <joint name="left_wheel_joint">
-                <command_interface name="velocity">
-                    <param name="min">-10</param>
-                    <param name="max">10</param>
-                </command_interface>
-                <state_interface name="velocity"/>
-                <state_interface name="position"/>
-            </joint>
-            <joint name="right_wheel_joint">
-                <command_interface name="velocity">
-                    <param name="min">-10</param>
-                    <param name="max">10</param>
-                </command_interface>
-                <state_interface name="velocity"/>
-                <state_interface name="position"/>
-            </joint>
-        </ros2_control>
-    </xacro:if>
+    <ros2_control name="GazeboSystem" type="system">
+        <hardware>
+            <plugin>gazebo_ros2_control/GazeboSystem</plugin>
+        </hardware>
+        <joint name="left_wheel_joint">
+            <command_interface name="velocity">
+                <param name="min">-10</param>
+                <param name="max">10</param>
+            </command_interface>
+            <state_interface name="velocity"/>
+            <state_interface name="position"/>
+        </joint>
+        <joint name="right_wheel_joint">
+            <command_interface name="velocity">
+                <param name="min">-10</param>
+                <param name="max">10</param>
+            </command_interface>
+            <state_interface name="velocity"/>
+            <state_interface name="position"/>
+        </joint>
+    </ros2_control>
     <gazebo>
         <plugin name="gazebo_ros2_control" filename="libgazebo_ros2_control.so">

Commit message: better wheels

File: src/boxbots/description/axeBot.xacro (robot description, xacro)
@@ -17,4 +17,13 @@
     <!-- BASE LINK -->
     <link name="base_link"></link>
+    <!-- BASE FOOTPRINT LINK -->
+    <!-- for 2d space reference. for mapping-->
+    <joint name="base_footprint_joint" type="fixed">
+        <parent link="base_link"/>
+        <child link="base_footprint"/>
+        <origin xyz="0 0 0" rpy="0 0 0"/>
+    </joint>
+    <link name="base_footprint">
+    </link>
     <!-- chassis -->
     <joint name="chassis_joint" type="fixed">
@@ -61,7 +70,7 @@
         </visual>
         <collision>
-            <origin xyz="0.287 -0.225 -0.1427" rpy="${pi/2} 0 ${pi/2}"/>
-            <geometry>
-                <mesh filename="file://$(find boxbots)/description/meshes/AxeBot/left_wheel.dae" scale="0.10 0.10 0.10"/>
+            <origin xyz="0 -0.03 0" rpy="${pi/2} 0 0"/>
+            <geometry>
+                <cylinder radius="0.1" length="0.05"/>
             </geometry>
         </collision>
@@ -90,7 +99,7 @@
         </visual>
         <collision>
-            <origin xyz="0.287 0.225 -0.1427" rpy="${pi/2} 0 ${pi/2}"/>
-            <geometry>
-                <mesh filename="file://$(find boxbots)/description/meshes/AxeBot/right_wheel.dae" scale="0.10 0.10 0.10"/>
+            <origin xyz="0 0.03 0" rpy="${pi/2} 0 0"/>
+            <geometry>
+                <cylinder radius="0.1" length="0.05"/>
             </geometry>
         </collision>
