Commit message: Modelo "Don barredora terminado"

File: src/boxbots/description/robot_core.xacro (robot description, xacro)
@@ -182,3 +182,30 @@
         <material>Gazebo/Black</material>
     </gazebo>
+    <!-- RAMP -->
+    <joint name="ramp_joint" type="fixed">
+        <parent link="chassis"/>
+        <child link="ramp"/>
+        <origin xyz="0.6 0 0.01"/>
+    </joint>
+    <link name="ramp">
+        <visual>
+            <geometry>
+                <mesh filename="file://$(find boxbots)/description/meshes/ramp1x1x1.dae" scale="0.24 0.4 0.2" />
+            </geometry>
+            <material name="black"/>2
+        </visual>
+        <collision>
+            <geometry>
+                <mesh filename="file://$(find boxbots)/description/meshes/ramp1x1x1.dae" scale="0.24 0.4 0.2" />
+            </geometry>
+        </collision>
+        <inertial>
+            <origin xyz="0.09909938 0.00000001 -0.00406687"/>
+            <mass value="1.00000000"/>
+            <inertia ixx="0.01520037" ixy="-0.00000000" ixz="0.00168628" iyy="0.00506596" iyz="0.00000000" izz="0.01653226"/>
+          </inertial>
+    </link>
+    <gazebo reference="lidar_support">
+        <material>Gazebo/Black</material>
+    </gazebo>
 </robot>

Commit message: color change fix dedazo

File: src/boxbots/description/robot_core.xacro (robot description, xacro)
@@ -32,5 +32,5 @@
                 <box size="0.6 0.4 0.2"/>
             </geometry>
-            <material name="white"/>
+            <material name="gray"/>
         </visual>
         <collision>
@@ -40,10 +40,10 @@
             </geometry>
         </collision>
-        <xacro:inertial_box mass="1" x="0.6" y="0.4" z="0.2">
+        <xacro:inertial_box mass="3" x="0.6" y="0.4" z="0.2">
             <origin xyz="0.3 0 0.1" rpy="0 0 0"/>
         </xacro:inertial_box>
     </link>
     <gazebo reference="chassis">
-        <material>Gazebo/White</material>
+        <material>Gazebo/Gray</material>
     </gazebo>
     <!--LEFT WHEEL LINK-->
@@ -60,5 +60,5 @@
                 <cylinder radius="0.1" length="0.05"/>
             </geometry>
-            <material name="blue"/>
+            <material name="black"/>
         </visual>
         <collision>
@@ -72,5 +72,5 @@
     </link>
     <gazebo reference="left_wheel">
-        <material>Gazebo/Blue</material>
+        <material>Gazebo/Black</material>
     </gazebo>
     <!--RIGHT WHEEL LINK-->
@@ -87,5 +87,5 @@
                 <cylinder radius="0.1" length="0.05"/>
             </geometry>
-            <material name="blue"/>
+            <material name="black"/>
         </visual>
         <collision>
@@ -99,5 +99,5 @@
     </link>
     <gazebo reference="right_wheel">
-        <material>Gazebo/Blue</material>
+        <material>Gazebo/Black</material>
     </gazebo>
     <!-- CASTER BASE LINK-->
@@ -193,5 +193,5 @@
                 <mesh filename="file://$(find boxbots)/description/meshes/ramp1x1x1.dae" scale="0.24 0.4 0.2" />
             </geometry>
-            <material name="black"/>2
+            <material name="gray"/>
         </visual>
         <collision>
@@ -206,6 +206,3 @@
           </inertial>
     </link>
-    <gazebo reference="lidar_support">
-        <material>Gazebo/Black</material>
-    </gazebo>
 </robot>

Commit message: SLAM y multiplex del nav

File: src/boxbots/description/robot_core.xacro (robot description, xacro)
@@ -29,4 +29,12 @@
     <link name="base_footprint">
     </link>
+    <!-- BASE_FOOTPRINT LINK -->
+    <joint name="base_footprint_joint" type="fixed">
+        <parent link="base_link"/>
+        <child link="base_footprint"/>
+        <origin xyz="0 0 0" rpy="0 0 0"/>
+    </joint>
+    <link name="base_footprint">
+    </link>
     <!-- CHASSIS LINK-->
     <joint name="chassis_joint" type="fixed">

Commit message: fix duplicated link base_footprint

File: src/boxbots/description/robot_core.xacro (robot description, xacro)
@@ -30,4 +30,5 @@
     </link>
     <!-- BASE_FOOTPRINT LINK -->
+<!--
     <joint name="base_footprint_joint" type="fixed">
         <parent link="base_link"/>
@@ -36,5 +37,5 @@
     </joint>
     <link name="base_footprint">
-    </link>
+    </link> -->
     <!-- CHASSIS LINK-->
     <joint name="chassis_joint" type="fixed">

Commit message: comment deleted

File: src/boxbots/description/robot_core.xacro (robot description, xacro)
@@ -29,13 +29,4 @@
     <link name="base_footprint">
     </link>
-    <!-- BASE_FOOTPRINT LINK -->
-<!--
-    <joint name="base_footprint_joint" type="fixed">
-        <parent link="base_link"/>
-        <child link="base_footprint"/>
-        <origin xyz="0 0 0" rpy="0 0 0"/>
-    </joint>
-    <link name="base_footprint">
-    </link> -->
     <!-- CHASSIS LINK-->
     <joint name="chassis_joint" type="fixed">
