Commit message: back to old topic remapping. New one doesnt work in xacro plugin

File: src/boxbots/description/imu.xacro (robot description, xacro)
@@ -16,6 +16,6 @@
           <plugin filename="libgazebo_ros_imu_sensor.so" name="imu_plugin">
             <ros>
-                <remap from="~/out" to="imu"/>
-                <namespace>/$(arg robot_name)</namespace>
+                <argument>~/out:=imu</argument>
+                <namespace>$(arg robot_name)</namespace>
             </ros>
             <bodyName>$(arg robot_name)/imu_link</bodyName>

File: src/boxbots/description/lidar.xacro (robot description, xacro)
@@ -2,6 +2,5 @@
 <robot xmlns:xacro="http://www.ros.org/wiki/xacro">
     <!-- Increase for more rays-->
-    <xacro:property name="horizontal_samples" value="1"/>
-    <xacro:property name="vertical_samples" value="1"/>
+    <xacro:property name="horizontal_resolution" value="1"/>
     <joint name="$(arg robot_name)/laser_joint" type="fixed">
         <parent link="$(arg robot_name)/lidar_support"/>
@@ -37,5 +36,5 @@
                     <horizontal>
                         <samples>180</samples>
-                        <resolution>${horizontal_samples}</resolution>
+                        <resolution>${horizontal_resolution}</resolution>
                         <min_angle>-1.57</min_angle>
                         <max_angle>1.57</max_angle>
@@ -43,5 +42,5 @@
                     <vertical>
                         <samples>1</samples>
-                        <resolution>${vertical_samples}</resolution>
+                        <resolution>1</resolution>
                         <min_angle>-0.06</min_angle>
                         <max_angle>0</max_angle>
@@ -55,6 +54,6 @@
             <plugin name="laser_controller" filename="libgazebo_ros_ray_sensor.so">
                 <ros>
-                    <remap from="~/out" to="scan"/>
-                    <namespace>/$(arg robot_name)</namespace>
+                    <argument>~/out:=imu</argument>
+                    <namespace>$(arg robot_name)</namespace>
                 </ros>
                 <output_type>sensor_msgs/LaserScan</output_type>
