Commit message: donBarredora colors modified

File: src/boxbots/description/donBarredora/donBarredora.xacro (robot description, xacro)
@@ -13,5 +13,5 @@
                 <mesh filename="file://$(find boxbots)/description/donBarredora/meshes/ramp1x1x1.dae" scale="0.24 0.4 0.2" />
             </geometry>
-            <material name="white"/>
+            <material name="black"/>
         </visual>
         <collision>
@@ -26,3 +26,6 @@
         </inertial>
     </link>
+    <gazebo reference="${robot_name}/ramp">
+        <material>Gazebo/Orange</material>
+    </gazebo>
 </robot>

File: src/boxbots/description/donBarredora/robot_core.xacro (robot description, xacro)
@@ -6,5 +6,5 @@
     </material>
     <material name="orange">
-        <color rgba="1 0.3 0.1 1"/>
+        <color rgba="1 0.5088 0.0468 1"/>
     </material>
     <material name="blue">
@@ -13,4 +13,7 @@
     <material name="black">
         <color rgba="0 0 0 1"/>
+    </material>
+    <material name="darkGrey">
+        <color rgba="0.175 0.175 0.175 1"/>
     </material>
     <material name="red">
@@ -41,5 +44,5 @@
                 <box size="0.6 0.4 0.2"/>
             </geometry>
-            <material name="orange"/>
+            <material name="darkGrey"/>
         </visual>
         <collision>
@@ -54,5 +57,5 @@
     </link>
     <gazebo reference="${robot_name}/chassis">
-        <material>Gazebo/Grey</material>
+        <material>Gazebo/DarkGrey</material>
     </gazebo>
     <!--LEFT WHEEL LINK-->
@@ -176,5 +179,5 @@
                 <cylinder radius="0.05" length="0.07"/>
             </geometry>
-            <material name="black"/>2
+            <material name="black"/>
         </visual>
         <collision>
