Commit message: color changes in robot_core

File: src/boxbots/description/donBarredora/robot_core.xacro (robot description, xacro)
@@ -16,4 +16,7 @@
     <material name="darkGrey">
         <color rgba="0.175 0.175 0.175 1"/>
+    </material>
+    <material name="grey">
+        <color rgba="0.3 0.3 0.3 1.0"/>
     </material>
     <material name="red">
@@ -44,5 +47,5 @@
                 <box size="0.6 0.4 0.2"/>
             </geometry>
-            <material name="darkGrey"/>
+            <material name="orange"/>
         </visual>
         <collision>
@@ -57,5 +60,5 @@
     </link>
     <gazebo reference="${robot_name}/chassis">
-        <material>Gazebo/DarkGrey</material>
+        <material>Gazebo/Orange</material>
     </gazebo>
     <!--LEFT WHEEL LINK-->
@@ -137,5 +140,5 @@
         </xacro:inertial_box>
     </link>
-    <gazebo reference="${robot_name}/caster_wheel">
+    <gazebo reference="${robot_name}/caster_base">
         <material>Gazebo/Black</material>
     </gazebo>
@@ -151,5 +154,5 @@
                 <sphere radius="0.02"/>
             </geometry>
-            <material name="black"/>
+            <material name="grey"/>
         </visual>
         <collision>
@@ -163,5 +166,5 @@
     </link>
     <gazebo reference="${robot_name}/caster_wheel">
-        <material>Gazebo/Black</material>
+        <material>Gazebo/Grey</material>
         <mu1 value="0.001"/>
         <mu2 value="0.001"/>

Commit message: cambios en los bots

File: src/boxbots/description/donBarredora/robot_core.xacro (robot description, xacro)
@@ -6,5 +6,5 @@
     </material>
     <material name="orange">
-        <color rgba="1 0.3 0.1 1"/>
+        <color rgba="1 0.5088 0.0468 1"/>
     </material>
     <material name="blue">
@@ -13,4 +13,10 @@
     <material name="black">
         <color rgba="0 0 0 1"/>
+    </material>
+    <material name="darkGrey">
+        <color rgba="0.175 0.175 0.175 1"/>
+    </material>
+    <material name="grey">
+        <color rgba="0.3 0.3 0.3 1.0"/>
     </material>
     <material name="red">
@@ -54,5 +60,5 @@
     </link>
     <gazebo reference="${robot_name}/chassis">
-        <material>Gazebo/Grey</material>
+        <material>Gazebo/Orange</material>
     </gazebo>
     <!--LEFT WHEEL LINK-->
@@ -134,5 +140,5 @@
         </xacro:inertial_box>
     </link>
-    <gazebo reference="${robot_name}/caster_wheel">
+    <gazebo reference="${robot_name}/caster_base">
         <material>Gazebo/Black</material>
     </gazebo>
@@ -148,5 +154,5 @@
                 <sphere radius="0.02"/>
             </geometry>
-            <material name="black"/>
+            <material name="grey"/>
         </visual>
         <collision>
@@ -160,5 +166,5 @@
     </link>
     <gazebo reference="${robot_name}/caster_wheel">
-        <material>Gazebo/Black</material>
+        <material>Gazebo/Grey</material>
         <mu1 value="0.001"/>
         <mu2 value="0.001"/>
@@ -176,5 +182,5 @@
                 <cylinder radius="0.05" length="0.07"/>
             </geometry>
-            <material name="black"/>2
+            <material name="black"/>
         </visual>
         <collision>

File: src/boxbots/description/lidar.xacro (robot description, xacro)
@@ -31,5 +31,5 @@
         <sensor name="laser" type="ray">
             <pose> 0 0 0 0 0 0 </pose>
-            <visualize>true</visualize>
+            <visualize>false</visualize>
             <update_rate>10</update_rate>
             <ray>
