Commit message: removiendo repetidos, removiendo tractor, Renombrando todas las partes según robot, Re nombrando topicos de publicación y namespaces, no funciona teleop ni funciona Lidar

File: src/boxbots/description/axeBot/axeBot.xacro (robot description, xacro)
@@ -1,5 +1,5 @@
 <?xml version="1.0"?>
 <robot xmlns:xacro="http://www.ros.org/wiki/xacro">
-    <xacro:include filename="inertial_macros.xacro"/>
+    <xacro:include filename="../inertial_macros.xacro"/>
     <material name="white">
         <color rgba="1 1 1 1"/>
@@ -14,26 +14,28 @@
         <color rgba="1 0.4 0.4 1"/>
     </material>
+    <xacro:arg name="robot_name" default="robot_core"/>
+    <xacro:property name="robot_name" value="$(arg robot_name)"/>
     <!-- BASE LINK -->
-    <link name="base_link"></link>
+    <link name="${robot_name}/base_link"></link>
     <!-- BASE FOOTPRINT LINK -->
     <!-- for 2d space reference. for mapping-->
-    <joint name="base_footprint_joint" type="fixed">
-        <parent link="base_link"/>
-        <child link="base_footprint"/>
+    <joint name="${robot_name}/base_footprint_joint" type="fixed">
+        <parent link="${robot_name}/base_link"/>
+        <child link="${robot_name}/base_footprint"/>
         <origin xyz="0 0 0" rpy="0 0 0"/>
     </joint>
-    <link name="base_footprint">
+    <link name="${robot_name}/base_footprint">
     </link>
     <!-- chassis -->
-    <joint name="chassis_joint" type="fixed">
-        <parent link="base_link"/>
-        <child link="chassis"/>
+    <joint name="${robot_name}/chassis_joint" type="fixed">
+        <parent link="${robot_name}/base_link"/>
+        <child link="${robot_name}/chassis"/>
         <origin xyz="0 0 0"/>
     </joint>
-    <link name="chassis">
+    <link name="${robot_name}/chassis">
         <visual>
             <origin xyz="0.3 0 -0.14" rpy="${pi/2} 0 ${pi/2}"/>
             <geometry>
-                <mesh filename="file://$(find boxbots)/description/meshes/AxeBot/chassis.dae" scale="0.10 0.10 0.10"/>
+                <mesh filename="file://$(find boxbots)/description/axeBot/meshes/chassis.dae" scale="0.10 0.10 0.10"/>
             </geometry>
             <material name="green"/>
@@ -42,5 +44,5 @@
             <origin xyz="0.3 0 -0.14" rpy="${pi/2} 0 ${pi/2}"/>
             <geometry>
-                <mesh filename="file://$(find boxbots)/description/meshes/AxeBot/chassis.dae" scale="0.09 0.1 0.1"/>
+                <mesh filename="file://$(find boxbots)/description/axeBot/meshes/chassis.dae" scale="0.09 0.1 0.1"/>
             </geometry>
         </collision>
@@ -49,20 +51,20 @@
         </xacro:inertial_box>
     </link>
-    <gazebo reference="chassis">
+    <gazebo reference="${robot_name}/chassis">
         <material>Gazebo/Turquoise</material>
     </gazebo>
     <!-- LEFT WHEEL -->
-    <joint name="left_wheel_joint" type="continuous">
-        <parent link="chassis"/>
-        <child link="left_wheel"/>
+    <joint name="${robot_name}/left_wheel_joint" type="continuous">
+        <parent link="${robot_name}/chassis"/>
+        <child link="${robot_name}/left_wheel"/>
         <!-- y=+(ancho/2+grosor_rueda/2)  -->
         <origin xyz="0 0.225 0"/>
         <axis xyz="0 1 0"/>
     </joint>
-    <link name="left_wheel">
+    <link name="${robot_name}/left_wheel">
         <visual>
             <origin xyz="0.287 -0.225 -0.1427" rpy="${pi/2} 0 ${pi/2}"/>
             <geometry>
-                <mesh filename="file://$(find boxbots)/description/meshes/AxeBot/left_wheel.dae" scale="0.10 0.10 0.10"/>
+                <mesh filename="file://$(find boxbots)/description/axeBot/meshes/left_wheel.dae" scale="0.10 0.10 0.10"/>
             </geometry>
             <material name="gray"/>
@@ -78,20 +80,20 @@
         </xacro:inertial_cylinder>
     </link>
-    <gazebo reference="left_wheel">
+    <gazebo reference="${robot_name}/left_wheel">
         <material>Gazebo/Gray</material>
     </gazebo>
     <!-- RIGHT WHEEL -->
-    <joint name="right_wheel_joint" type="continuous">
-        <parent link="chassis"/>
-        <child link="right_wheel"/>
+    <joint name="${robot_name}/right_wheel_joint" type="continuous">
+        <parent link="${robot_name}/chassis"/>
+        <child link="${robot_name}/right_wheel"/>
         <!-- y=-(ancho/2+grosor_rueda/2)  -->
         <origin xyz="0 -0.225 0"/>
         <axis xyz="0 1 0"/>
     </joint>
-    <link name="right_wheel">
+    <link name="${robot_name}/right_wheel">
         <visual>
             <origin xyz="0.287 0.225 -0.1427" rpy="${pi/2} 0 ${pi/2}"/>
             <geometry>
-                <mesh filename="file://$(find boxbots)/description/meshes/AxeBot/right_wheel.dae" scale="0.10 0.10 0.10"/>
+                <mesh filename="file://$(find boxbots)/description/axeBot/meshes/right_wheel.dae" scale="0.10 0.10 0.10"/>
             </geometry>
             <material name="gray"/>
@@ -107,18 +109,18 @@
         </xacro:inertial_cylinder>
     </link>
-    <gazebo reference="right_wheel">
+    <gazebo reference="${robot_name}/right_wheel">
         <material>Gazebo/Gray</material>
     </gazebo>
     <!-- BALL WHEEL -->
-    <joint name="caster_wheel_joint" type="fixed">
-        <parent link="chassis"/>
-        <child link="caster_wheel"/>
+    <joint name="${robot_name}/caster_wheel_joint" type="fixed">
+        <parent link="${robot_name}/chassis"/>
+        <child link="${robot_name}/caster_wheel"/>
         <origin xyz="0.36 0 -0.045"/>
     </joint>
-    <link name="caster_wheel">
+    <link name="${robot_name}/caster_wheel">
         <visual>
             <origin xyz="-0.06 0 -0.09" rpy="${pi/2} 0 ${pi/2}"/>
             <geometry>
-                <mesh filename="file://$(find boxbots)/description/meshes/AxeBot/ball_wheel.dae" scale="0.10 0.10 0.10"/>
+                <mesh filename="file://$(find boxbots)/description/axeBot/meshes/ball_wheel.dae" scale="0.10 0.10 0.10"/>
             </geometry>
             <material name="white"/>
@@ -127,5 +129,5 @@
             <origin xyz="-0.06 0 -0.09" rpy="${pi/2} 0 ${pi/2}"/>
             <geometry>
-                <mesh filename="file://$(find boxbots)/description/meshes/AxeBot/ball_wheel.dae" scale="0.10 0.10 0.10"/>
+                <mesh filename="file://$(find boxbots)/description/axeBot/meshes/ball_wheel.dae" scale="0.10 0.10 0.10"/>
             </geometry>
         </collision>
@@ -134,5 +136,5 @@
         </xacro:inertial_sphere>
     </link>
-    <gazebo reference="caster_wheel">
+    <gazebo reference="${robot_name}/caster_wheel">
         <material>Gazebo/White</material>
         <mu1 value="0.001"/>
@@ -140,14 +142,14 @@
     </gazebo>
     <!-- TAIL -->
-    <joint name="tail_joint" type="fixed">
-        <parent link="chassis"/>
-        <child link="tail"/>
+    <joint name="${robot_name}/tail_joint" type="fixed">
+        <parent link="${robot_name}/chassis"/>
+        <child link="${robot_name}/tail"/>
         <origin xyz="-0.15 0 0.25"/>
     </joint>
-    <link name="tail">
+    <link name="${robot_name}/tail">
         <visual>
             <origin xyz="0.4 0 -0.43" rpy="${pi/2} 0 ${pi/2}"/>
             <geometry>
-                <mesh filename="file://$(find boxbots)/description/meshes/AxeBot/tail.dae" scale="0.10 0.10 0.10"/>
+                <mesh filename="file://$(find boxbots)/description/axeBot/meshes/tail.dae" scale="0.10 0.10 0.10"/>
             </geometry>
             <material name="white"/>
@@ -156,5 +158,5 @@
             <origin xyz="0.4 0 -0.43" rpy="${pi/2} 0 ${pi/2}"/>
             <geometry>
-                <mesh filename="file://$(find boxbots)/description/meshes/AxeBot/tail.dae" scale="0.10 0.10 0.10"/>
+                <mesh filename="file://$(find boxbots)/description/axeBot/meshes/tail.dae" scale="0.10 0.10 0.10"/>
             </geometry>
         </collision>
@@ -163,18 +165,18 @@
         </xacro:inertial_box>
     </link>
-    <gazebo reference="tail">
+    <gazebo reference="${robot_name}/tail">
         <material>Gazebo/YellowGlow</material>
     </gazebo>
     <!-- AXE -->
-    <joint name="axe_joint" type="fixed">
-        <parent link="chassis"/>
-        <child link="axe"/>
+    <joint name="${robot_name}/axe_joint" type="fixed">
+        <parent link="${robot_name}/chassis"/>
+        <child link="${robot_name}/axe"/>
         <origin xyz="0.6 0 0.01" />
     </joint>
-    <link name="axe">
+    <link name="${robot_name}/axe">
         <visual>
             <origin xyz="-0.3 0 -0.15" rpy="${pi/2} 0 ${pi/2}"/>
             <geometry>
-                <mesh filename="file://$(find boxbots)/description/meshes/AxeBot/axe.dae" scale="0.10 0.10 0.10"/>
+                <mesh filename="file://$(find boxbots)/description/axeBot/meshes/axe.dae" scale="0.10 0.10 0.10"/>
             </geometry>
             <material name="red"/>
@@ -183,5 +185,5 @@
             <origin xyz="-0.3 0 -0.15" rpy="${pi/2} 0 ${pi/2}"/>
             <geometry>
-                <mesh filename="file://$(find boxbots)/description/meshes/AxeBot/axe.dae" scale="0.10 0.10 0.10"/>
+                <mesh filename="file://$(find boxbots)/description/axeBot/meshes/axe.dae" scale="0.10 0.10 0.10"/>
             </geometry>
         </collision>
@@ -190,14 +192,14 @@
         </xacro:inertial_box>
     </link>
-    <gazebo reference="axe">
+    <gazebo reference="${robot_name}/axe">
         <material>Gazebo/RedGlow</material>
     </gazebo>
     <!-- LIDAR SUPPORT LINK-->
-    <joint name="lidar_support_joint" type="fixed">
-        <parent link="tail"/>
-        <child link="lidar_support"/>
+    <joint name="${robot_name}/lidar_support_joint" type="fixed">
+        <parent link="${robot_name}/tail"/>
+        <child link="${robot_name}/lidar_support"/>
         <origin xyz="-0.07 0 0"/>
     </joint>
-    <link name="lidar_support">
+    <link name="${robot_name}/lidar_support">
         <visual>
             <origin xyz="0 0 0.035"/>
@@ -217,5 +219,5 @@
         </xacro:inertial_cylinder>
     </link>
-    <gazebo reference="lidar_support">
+    <gazebo reference="${robot_name}/lidar_support">
         <material>Gazebo/Black</material>
     </gazebo>

File: src/boxbots/description/donBarredora/donBarredora.xacro (robot description, xacro)
@@ -3,19 +3,19 @@
     <xacro:include filename="robot_core.xacro"/>
     <!-- RAMP -->
-    <joint name="ramp_joint" type="fixed">
-        <parent link="chassis"/>
-        <child link="ramp"/>
+    <joint name="${robot_name}/ramp_joint" type="fixed">
+        <parent link="${robot_name}/chassis"/>
+        <child link="${robot_name}/ramp"/>
         <origin xyz="0.6 0 0.01"/>
     </joint>
-    <link name="ramp">
+    <link name="${robot_name}/ramp">
         <visual>
             <geometry>
-                <mesh filename="file://$(find boxbots)/description/meshes/ramp1x1x1.dae" scale="0.24 0.4 0.2" />
+                <mesh filename="file://$(find boxbots)/description/donBarredora/meshes/ramp1x1x1.dae" scale="0.24 0.4 0.2" />
             </geometry>
-            <material name="gray"/>
+            <material name="white"/>
         </visual>
         <collision>
             <geometry>
-                <mesh filename="file://$(find boxbots)/description/meshes/ramp1x1x1.dae" scale="0.24 0.4 0.2" />
+                <mesh filename="file://$(find boxbots)/description/donBarredora/meshes/ramp1x1x1.dae" scale="0.24 0.4 0.2" />
             </geometry>
         </collision>

File: src/boxbots/description/donBarredora/robot_core.xacro (robot description, xacro)
@@ -1,5 +1,5 @@
 <?xml version="1.0"?>
 <robot xmlns:xacro="http://www.ros.org/wiki/xacro">
-    <xacro:include filename="inertial_macros.xacro"/>
+    <xacro:include filename="../inertial_macros.xacro"/>
     <material name="white">
         <color rgba="1 1 1 1"/>
@@ -17,23 +17,23 @@
         <color rgba="1 0 0 1"/>
     </material>
+    <xacro:arg name="robot_name" default="robot_core"/>
+    <xacro:property name="robot_name" value="$(arg robot_name)"/>
     <!-- BASE LINK -->
-    <link name="base_link">
-    </link>
+    <link name="${robot_name}/base_link"></link>
     <!-- BASE FOOTPRINT LINK -->
     <!-- for 2d space reference. for mapping-->
-    <joint name="base_footprint_joint" type="fixed">
-        <parent link="base_link"/>
-        <child link="base_footprint"/>
+    <joint name="${robot_name}/base_footprint_joint" type="fixed">
+        <parent link="${robot_name}/base_link"/>
+        <child link="${robot_name}/base_footprint"/>
         <origin xyz="0 0 0" rpy="0 0 0"/>
     </joint>
-    <link name="base_footprint">
-    </link>
+    <link name="${robot_name}/base_footprint"></link>
     <!-- CHASSIS LINK-->
-    <joint name="chassis_joint" type="fixed">
-        <parent link="base_link"/>
-        <child link="chassis"/>
+    <joint name="${robot_name}/chassis_joint" type="fixed">
+        <parent link="${robot_name}/base_link"/>
+        <child link="${robot_name}/chassis"/>
         <origin xyz="-0.15 0 -0.05"/>
     </joint>
-    <link name="chassis">
+    <link name="${robot_name}/chassis">
         <visual>
             <origin xyz="0.3 0 0.1"/>
@@ -41,5 +41,5 @@
                 <box size="0.6 0.4 0.2"/>
             </geometry>
-            <material name="grey"/>
+            <material name="orange"/>
         </visual>
         <collision>
@@ -53,16 +53,16 @@
         </xacro:inertial_box>
     </link>
-    <gazebo reference="chassis">
+    <gazebo reference="${robot_name}/chassis">
         <material>Gazebo/Grey</material>
     </gazebo>
     <!--LEFT WHEEL LINK-->
-    <joint name="left_wheel_joint" type="continuous">
-        <parent link="base_link"/>
-        <child link="left_wheel"/>
+    <joint name="${robot_name}/left_wheel_joint" type="continuous">
+        <parent link="${robot_name}/base_link"/>
+        <child link="${robot_name}/left_wheel"/>
         <!-- y=+(ancho/2+grosor_rueda/2)  -->
         <origin xyz="0 0.225 0" rpy="-${pi/2} 0 0"/>
         <axis xyz="0 0 1"/>
     </joint>
-    <link name="left_wheel">
+    <link name="${robot_name}/left_wheel">
         <visual>
             <geometry>
@@ -80,16 +80,16 @@
         </xacro:inertial_cylinder>
     </link>
-    <gazebo reference="left_wheel">
+    <gazebo reference="${robot_name}/left_wheel">
         <material>Gazebo/Black</material>
     </gazebo>
     <!--RIGHT WHEEL LINK-->
-    <joint name="right_wheel_joint" type="continuous">
-        <parent link="base_link"/>
-        <child link="right_wheel"/>
+    <joint name="${robot_name}/right_wheel_joint" type="continuous">
+        <parent link="${robot_name}/base_link"/>
+        <child link="${robot_name}/right_wheel"/>
         <!-- y=-(ancho/2+grosor_rueda/2)  -->
         <origin xyz="0 -0.225 0" rpy="${pi/2} 0 0"/>
         <axis xyz="0 0 -1"/>
     </joint>
-    <link name="right_wheel">
+    <link name="${robot_name}/right_wheel">
         <visual>
             <geometry>
@@ -107,14 +107,14 @@
         </xacro:inertial_cylinder>
     </link>
-    <gazebo reference="right_wheel">
+    <gazebo reference="${robot_name}/right_wheel">
         <material>Gazebo/Black</material>
     </gazebo>
     <!-- CASTER BASE LINK-->
-    <joint name="caster_base_joint" type="fixed">
-        <parent link="chassis"/>
-        <child link="caster_base"/>
+    <joint name="${robot_name}/caster_base_joint" type="fixed">
+        <parent link="${robot_name}/chassis"/>
+        <child link="${robot_name}/caster_base"/>
         <origin xyz="0.5 0 0"/>
     </joint>
-    <link name="caster_base">
+    <link name="${robot_name}/caster_base">
         <visual>
             <origin xyz="0 0 -0.015"/>
@@ -134,14 +134,14 @@
         </xacro:inertial_box>
     </link>
-    <gazebo reference="caster_wheel">
+    <gazebo reference="${robot_name}/caster_wheel">
         <material>Gazebo/Black</material>
     </gazebo>
     <!-- CASTER WHEEL LINK-->
-    <joint name="caster_wheel_joint" type="fixed">
-        <parent link="caster_base"/>
-        <child link="caster_wheel"/>
+    <joint name="${robot_name}/caster_wheel_joint" type="fixed">
+        <parent link="${robot_name}/caster_base"/>
+        <child link="${robot_name}/caster_wheel"/>
         <origin xyz="0 0 -0.03"/>
     </joint>
-    <link name="caster_wheel">
+    <link name="${robot_name}/caster_wheel">
         <visual>
             <geometry>
@@ -159,5 +159,5 @@
         </xacro:inertial_sphere>
     </link>
-    <gazebo reference="caster_wheel">
+    <gazebo reference="${robot_name}/caster_wheel">
         <material>Gazebo/Black</material>
         <mu1 value="0.001"/>
@@ -165,10 +165,10 @@
     </gazebo>
     <!-- LIDAR SUPPORT LINK-->
-    <joint name="lidar_support_joint" type="fixed">
-        <parent link="chassis"/>
-        <child link="lidar_support"/>
+    <joint name="${robot_name}/lidar_support_joint" type="fixed">
+        <parent link="${robot_name}/chassis"/>
+        <child link="${robot_name}/lidar_support"/>
         <origin xyz="0.15 0 0.2"/>
     </joint>
-    <link name="lidar_support">
+    <link name="${robot_name}/lidar_support">
         <visual>
             <origin xyz="0 0 0.035"/>
@@ -188,5 +188,5 @@
         </xacro:inertial_cylinder>
     </link>
-    <gazebo reference="lidar_support">
+    <gazebo reference="${robot_name}/lidar_support">
         <material>Gazebo/Black</material>
     </gazebo>

File: src/boxbots/description/gazebo_control.xacro (robot description, xacro)
@@ -1,10 +1,15 @@
 <?xml version="1.0"?>
 <robot xmlns:xacro="http://www.ros.org/wiki/xacro">
+    <xacro:arg name="robot_name" default="robot_core"/>
+    <xacro:property name="robot_name" value="$(arg robot_name)"/>
     <gazebo>
         <plugin name="diff_drive" filename="libgazebo_ros_diff_drive.so">
+            <ros>
+                <namespace>/$(arg robot_name)</namespace>
+            </ros>
             <!-- Wheel Information -->
-            <left_joint>left_wheel_joint</left_joint>
-            <right_joint>right_wheel_joint</right_joint>
-            <wheel_separation>0.45</wheel_separation>
+            <left_joint>$(arg robot_name)/left_wheel_joint</left_joint>
+            <right_joint>$(arg robot_name)/right_wheel_joint</right_joint>
+            <wheel_separation>0.4</wheel_separation>
             <wheel_diameter>0.2</wheel_diameter>
             <!-- Limits -->
@@ -13,5 +18,5 @@
             <!-- Output -->
             <odometry_frame>odom</odometry_frame>
-            <robot_base_frame>base_link</robot_base_frame>
+            <robot_base_frame>$(arg robot_name)/base_link</robot_base_frame>
             <publish_odom>true</publish_odom>
             <publish_odom_tf>true</publish_odom_tf>

File: src/boxbots/description/imu.xacro (robot description, xacro)
@@ -1,13 +1,13 @@
 <?xml version="1.0"?>
 <robot xmlns:xacro="http://www.ros.org/wiki/xacro">
-    <joint name="imu_joint" type="fixed">
-        <parent link="base_link"/>
-        <child link="imu_link"/>
+    <joint name="$(arg robot_name)/imu_joint" type="fixed">
+        <parent link="$(arg robot_name)/base_link"/>
+        <child link="$(arg robot_name)/imu_link"/>
         <axis xyz="1 0 0" />
     </joint>
-    <link name="imu_link"/>
-    <gazebo reference="imu_link">
+    <link name="$(arg robot_name)/imu_link"/>
+    <gazebo reference="$(arg robot_name)/imu_link">
         <gravity>true</gravity>
-        <sensor name="imu_sensor" type="imu">
+        <sensor name="$(arg robot_name)/imu_sensor" type="imu">
           <always_on>true</always_on>
           <update_rate>100</update_rate>
@@ -16,12 +16,13 @@
           <plugin filename="libgazebo_ros_imu_sensor.so" name="imu_plugin">
             <ros>
-                <argument>~/out:=imu</argument>
+                <remap from="~/out" to="imu"/>
+                <namespace>/$(arg robot_name)</namespace>
             </ros>
-            <bodyName>imu_link</bodyName>
+            <bodyName>$(arg robot_name)/imu_link</bodyName>
             <updateRateHZ>10.0</updateRateHZ>
             <gaussianNoise>0.0</gaussianNoise>
             <xyzOffset>0 0 0</xyzOffset>
             <rpyOffset>0 0 0</rpyOffset>
-            <frameName>imu_link</frameName>
+            <frameName>$(arg robot_name)/imu_link</frameName>
             <initialOrientationAsReference>false</initialOrientationAsReference>
           </plugin>

File: src/boxbots/description/lidar.xacro (robot description, xacro)
@@ -1,10 +1,13 @@
 <?xml version="1.0"?>
 <robot xmlns:xacro="http://www.ros.org/wiki/xacro">
-    <joint name="laser_joint" type="fixed">
-        <parent link="lidar_support"/>
-        <child link="laser_frame"/>
+    <!-- Increase for more rays-->
+    <xacro:property name="horizontal_samples" value="1"/>
+    <xacro:property name="vertical_samples" value="1"/>
+    <joint name="$(arg robot_name)/laser_joint" type="fixed">
+        <parent link="$(arg robot_name)/lidar_support"/>
+        <child link="$(arg robot_name)/laser_frame"/>
         <origin xyz="0 0 0.07" rpy="0 0 0"/>
     </joint>
-    <link name="laser_frame">
+    <link name="$(arg robot_name)/laser_frame">
         <visual>
             <origin xyz="0 0 0.015" rpy="0 0 0"/>
@@ -24,16 +27,17 @@
         </xacro:inertial_cylinder>
     </link>
-    <gazebo reference="laser_frame">
+    <gazebo reference="$(arg robot_name)/laser_frame">
         <material>Gazebo/Red</material>
         <sensor name="laser" type="ray">
             <pose> 0 0 0 0 0 0 </pose>
-            <visualize>false</visualize>
+            <visualize>true</visualize>
             <update_rate>10</update_rate>
             <ray>
                 <scan>
                     <horizontal>
-                        <samples>360</samples>
-                        <min_angle>-3.14</min_angle>
-                        <max_angle>3.14</max_angle>
+                        <samples>180</samples>
+                        <resolution>${horizontal_samples}</resolution>
+                        <min_angle>-1.57</min_angle>
+                        <max_angle>1.57</max_angle>
                     </horizontal>
                 </scan>
@@ -45,8 +49,9 @@
             <plugin name="laser_controller" filename="libgazebo_ros_ray_sensor.so">
                 <ros>
-                    <argument>~/out:=scan</argument>
+                    <remap from="~/out" to="scan"/>
+                    <namespace>/$(arg robot_name)</namespace>
                 </ros>
                 <output_type>sensor_msgs/LaserScan</output_type>
-                <frame_name>laser_frame</frame_name>
+                <frame_name>$(arg robot_name)/laser_frame</frame_name>
             </plugin>
         </sensor>
