Commit message: removiendo repetidos, removiendo tractor, Renombrando todas las partes según robot, Re nombrando topicos de publicación y namespaces, no funciona teleop ni funciona Lidar

File: src/boxbots/description/robot.urdf.xacro (robot description, xacro)
@@ -3,11 +3,6 @@
     <xacro:arg name="robot_name" default="robot_core"/>
     <xacro:property name="robot_name" value="$(arg robot_name)"/>
-    <xacro:include filename="${robot_name}.xacro"/>
-    <xacro:if value="$(arg use_ros2_control)">
-        <xacro:include filename="ros2_control.xacro" />
-    </xacro:if>
-    <xacro:unless value="$(arg use_ros2_control)">
-        <xacro:include filename="gazebo_control.xacro" />
-    </xacro:unless>
+    <xacro:include filename="${robot_name}/${robot_name}.xacro"/>
+    <xacro:include filename="gazebo_control.xacro" />
     <xacro:include filename="lidar.xacro"/>
     <xacro:include filename="imu.xacro"/>

Commit message: Lidares a la misma altura

File: src/boxbots/description/axeBot/axeBot.xacro (robot description, xacro)
@@ -199,5 +199,5 @@
         <parent link="${robot_name}/tail"/>
         <child link="${robot_name}/lidar_support"/>
-        <origin xyz="-0.07 0 0"/>
+        <origin xyz="0.2 0 -0.1"/>
     </joint>
     <link name="${robot_name}/lidar_support">

File: src/boxbots/description/lidar.xacro (robot description, xacro)
@@ -41,4 +41,10 @@
                         <max_angle>1.57</max_angle>
                     </horizontal>
+                    <vertical>
+                        <samples>1</samples>
+                        <resolution>${vertical_samples}</resolution>
+                        <min_angle>-0.06</min_angle>
+                        <max_angle>0</max_angle>
+                    </vertical>
                 </scan>
                 <range>
